Commit message: update 2026-08-18_14:55:37

File: x3plus_description/urdf/yahboomcar_X3plus.urdf (robot description, URDF)
Before this commit: robot yahboomcar_X3plus, 21 links, 20 joints
Links:
- link arm_link1: geometry collision mesh filename=package://meshes/X3plus/collision/arm_link1.obj; visual mesh filename=package://meshes/X3plus/visual/arm_link1.obj
- link arm_link2: geometry collision mesh filename=package://meshes/X3plus/collision/arm_link2.obj; visual mesh filename=package://meshes/X3plus/visual/arm_link2.obj
- link arm_link3: geometry collision mesh filename=package://meshes/X3plus/collision/arm_link3.obj; visual mesh filename=package://meshes/X3plus/visual/arm_link3.obj
- link arm_link4: geometry collision mesh filename=package://meshes/X3plus/collision/arm_link4.obj; visual mesh filename=package://meshes/X3plus/visual/arm_link4.obj
- link arm_link5: geometry collision mesh filename=package://meshes/X3plus/collision/arm_link5.obj; visual mesh filename=package://meshes/X3plus/visual/arm_link5.obj
- link back_left_wheel: geometry collision mesh filename=package://meshes/X3plus/collision/back_left_wheel.obj; visual mesh filename=package://meshes/X3plus/visual/back_left_wheel.obj
- link back_right_wheel: geometry collision mesh filename=package://meshes/X3plus/collision/back_right_wheel.obj; visual mesh filename=package://meshes/X3plus/visual/back_right_wheel.obj
- link base_link: geometry collision mesh filename=package://meshes/X3plus/collision/base_link_wo_wheels.obj; visual mesh filename=package://meshes/X3plus/visual/base_link_wo_wheels.obj
- link camera_link: geometry collision mesh filename=package://meshes/sensor/collision/camera_link.obj; visual mesh filename=package://meshes/sensor/visual/camera_link.obj
- link front_left_wheel: geometry collision mesh filename=package://meshes/X3plus/collision/front_left_wheel.obj; visual mesh filename=package://meshes/X3plus/visual/front_left_wheel.obj
- link front_right_wheel: geometry collision mesh filename=package://meshes/X3plus/collision/front_right_wheel.obj; visual mesh filename=package://meshes/X3plus/visual/front_right_wheel.obj
- link laser_link: geometry collision mesh filename=package://meshes/sensor/collision/laser_link.obj; visual mesh filename=package://meshes/sensor/visual/laser_link.obj
- link llink1: geometry collision mesh filename=package://meshes/X3plus/visual/llink1.obj; visual mesh filename=package://meshes/X3plus/visual/llink1.obj
- link llink2: geometry collision mesh filename=package://meshes/X3plus/visual/llink2.obj; visual mesh filename=package://meshes/X3plus/visual/llink2.obj
- link llink3: geometry collision mesh filename=package://meshes/X3plus/visual/llink3.obj; visual mesh filename=package://meshes/X3plus/visual/llink3.obj
- link mono_link: geometry collision mesh filename=package://meshes/sensor/collision/mono_link.obj; visual mesh filename=package://meshes/sensor/visual/mono_link.obj
- link rlink1: geometry collision mesh filename=package://meshes/X3plus/visual/rlink1.obj; visual mesh filename=package://meshes/X3plus/visual/rlink1.obj
- link rlink2: geometry collision mesh filename=package://meshes/X3plus/visual/rlink2.obj; visual mesh filename=package://meshes/X3plus/visual/rlink2.obj
- link rlink3: geometry collision mesh filename=package://meshes/X3plus/visual/rlink3.obj; visual mesh filename=package://meshes/X3plus/visual/rlink3.obj
